File: lm393_ldr_save_rocket.kicad_sch (KiCad schematic)
At the start: 15 parts, among them J1 BAT 9V, J2 IGNITER, Q1 TIP122, U1 LM7805, U2 LM393

Commit message: ajustes de posicionamento de componentes na placa
Parts:
- removed Q1: TIP122, Package_TO_SOT_THT:TO-220-3_Horizontal_TabDown, symbol Transistor_BJT:TIP122
- added Q2: TIP120, Package_TO_SOT_THT:TO-220-3_Horizontal_TabDown, symbol Transistor_BJT:TIP120
Connections:
- net at R4.2: now also Q2.1 (B)
- net at C1.1, J1.1 (Pin_1), U1.1 (VI): now also Q2.2 (C)
- net at J2.1 (Pin_1): now also Q2.3 (E)

Commit message: jumper de segurança
Parts:
- added J3: JUMP, Button_Switch_THT:SW_DIP_SPSTx01_Slide_6.7x4.1mm_W7.62mm_P2.54mm_LowProfile, symbol Connector_Generic:Conn_01x02
Connections:
- net at Q2.3 (E): now also J3.1 (Pin_1); no longer J2.1 (Pin_1)
- new net: J2.1 (Pin_1), J3.2 (Pin_2)
Other:
- moved on the sheet: J2
Changed lines of the file:
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@@
+	(wire
+		(pts
+			(xy 29.21 69.85) (xy 151.13 69.85)
+		)
+		(stroke
+			(width 0)
+			(type default)
+		)
+	)
 	(wire
 		(pts
@@
 	(wire
 		(pts
+			(xy 151.13 67.31) (xy 157.48 67.31)
+		)
+		(stroke
+			(width 0)
+			(type default)
+		)
+	)
+	(wire
+		(pts
 			(xy 29.21 21.59) (xy 171.45 21.59)
 		)
@@
 	(wire
 		(pts
+			(xy 160.02 67.31) (xy 171.45 67.31)
+		)
+		(stroke
+			(width 0)
+			(type default)
+		)
+	)
+	(wire
+		(pts
 			(xy 73.66 58.42) (xy 73.66 52.07)
 		)
@@
 	(wire
 		(pts
+			(xy 171.45 53.34) (xy 171.45 59.69)
+		)
+		(stroke
+			(width 0)
+			(type default)
+		)
+	)
+	(wire
+		(pts
 			(xy 29.21 38.1) (xy 29.21 45.72)
 		)
@@
 	(wire
 		(pts
+			(xy 151.13 69.85) (xy 151.13 67.31)
+		)
+		(stroke
+			(width 0)
+			(type default)
+		)
+	)
+	(wire
+		(pts
 			(xy 129.54 63.5) (xy 134.62 63.5)
 		)
@@
 	(wire
 		(pts
-			(xy 171.45 53.34) (xy 171.45 58.42)
+			(xy 171.45 67.31) (xy 171.45 62.23)
 		)
 		(stroke
@@
 	(wire
 		(pts
-			(xy 29.21 69.85) (xy 171.45 69.85)
-		)
-		(stroke
-			(width 0)
-			(type default)
-		)
-	)
-	(wire
-		(pts
 			(xy 73.66 38.1) (xy 73.66 27.94)
-		)
-		(stroke
-			(width 0)
-			(type default)
-		)
-	)
-	(wire
-		(pts
-			(xy 171.45 69.85) (xy 171.45 60.96)
 		)
 		(stroke
@@
 	)
 	(symbol
+		(lib_id "Connector_Generic:Conn_01x02")
+		(at 176.53 59.69 0)
+		(unit 1)
+		(exclude_from_sim no)
+		(in_bom yes)
+		(on_board yes)
+		(dnp no)
+		(fields_autoplaced yes)
+		(property "Reference" "J3"
+			(at 179.07 59.6899 0)
+			(effects
+				(font
+					(size 1.27 1.27)
+				)
+				(justify left)
+			)
+		)
+		(property "Value" "JUMP"
+			(at 179.07 62.2299 0)
+			(effects
+				(font
+					(size 1.27 1.27)
+				)
+				(justify left)
+			)
+		)
+		(property "Footprint" "Button_Switch_THT:SW_DIP_SPSTx01_Slide_6.7x4.1mm_W7.62mm_P2.54mm_LowProfile"
+			(at 176.53 59.69 0)
+			(effects
+				(font
+					(size 1.27 1.27)
+				)
+				(hide yes)
+			)
+		)
+		(property "Datasheet" "~"
+			(at 176.53 59.69 0)
+			(effects
+				(font
+					(size 1.27 1.27)
+				)
+				(hide yes)
+			)
+		)
+		(property "Description" "Generic connector, single row, 01x02, script generated (kicad-library-utils/schlib/autogen/connector/)"
+			(at 176.53 59.69 0)
+			(effects
+				(font
+					(size 1.27 1.27)
+				)
+				(hide yes)
+			)
+		)
+		(pin "2"
+		)
+		(pin "1"
+		)
+		(instances
+			(project "lm393_ldr_save_rocket"
+				(path "/ae093865-4f5b-4e6d-9eba-48d65543423e"
+					(reference "J3")
+					(unit 1)
+				)
+			)
+		)
+	)
+	(symbol
 		(lib_id "Device:R")
 		(at 146.05 36.83 0)
@@
 	(symbol
 		(lib_id "Connector_Generic:Conn_01x02")
-		(at 176.53 58.42 0)
+		(at 160.02 72.39 270)
 		(unit 1)
 		(exclude_from_sim no)
@@
 		(fields_autoplaced yes)
 		(property "Reference" "J2"
-			(at 179.07 58.4199 0)
+			(at 162.56 71.1199 90)
 			(effects
 				(font
@@
 		)
 		(property "Value" "IGNITER"
-			(at 179.07 60.9599 0)
+			(at 162.56 73.6599 90)
 			(effects
 				(font
@@
 		)
 		(property "Footprint" "TerminalBlock_Phoenix:TerminalBlock_Phoenix_MKDS-1,5-2-5.08_1x02_P5.08mm_Horizontal"
-			(at 176.53 58.42 0)
+			(at 160.02 72.39 0)
 			(effects
 				(font
@@
 		)
 		(property "Datasheet" "~"
-			(at 176.53 58.42 0)
+			(at 160.02 72.39 0)
 			(effects
 				(font
@@
 		)
 		(property "Description" "Generic connector, single row, 01x02, script generated (kicad-library-utils/schlib/autogen/connector/)"
-			(at 176.53 58.42 0)
-			(effects
-				(font
+			(at 160.02 72.39 0)
+			(effects
+				(font

Commit message: posicionamento carga tip120
Parts:
- R4: value 4k7 -> 470
- R5: value 470 -> 220
Connections:
- net GND: now also Q2.3 (E); no longer J2.2 (Pin_2)
- net VCC: now also R5.1
- net at R3.2, R4.1, U2.1: no longer R5.1
- net at C1.1, J1.1 (Pin_1), U1.1 (VI): now also J3.1 (Pin_1); no longer Q2.2 (C)
- new net: J2.2 (Pin_2), Q2.2 (C)
Other:
- moved on the sheet: J2, J3
Changed lines of the file:
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@@
+	)
+	(junction
+		(at 140.97 27.94)
+		(diameter 0)
+		(color 0 0 0 0)
 	)
 	(junction
@@
 	(wire
 		(pts
-			(xy 129.54 27.94) (xy 146.05 27.94)
-		)
-		(stroke
-			(width 0)
-			(type default)
-		)
-	)
-	(wire
-		(pts
-			(xy 29.21 69.85) (xy 151.13 69.85)
+			(xy 129.54 27.94) (xy 140.97 27.94)
 		)
 		(stroke
@@
 	(wire
 		(pts
-			(xy 146.05 48.26) (xy 146.05 52.07)
+			(xy 140.97 27.94) (xy 140.97 52.07)
 		)
 		(stroke
@@
 	(wire
 		(pts
-			(xy 151.13 67.31) (xy 157.48 67.31)
-		)
-		(stroke
-			(width 0)
-			(type default)
-		)
-	)
-	(wire
-		(pts
 			(xy 29.21 21.59) (xy 171.45 21.59)
 		)
@@
 	(wire
 		(pts
-			(xy 160.02 67.31) (xy 171.45 67.31)
-		)
-		(stroke
-			(width 0)
-			(type default)
-		)
-	)
-	(wire
-		(pts
 			(xy 73.66 58.42) (xy 73.66 52.07)
 		)
@@
 	(wire
 		(pts
-			(xy 171.45 53.34) (xy 171.45 59.69)
-		)
-		(stroke
-			(width 0)
-			(type default)
-		)
-	)
-	(wire
-		(pts
 			(xy 29.21 38.1) (xy 29.21 45.72)
 		)
@@
 	(wire
 		(pts
-			(xy 151.13 69.85) (xy 151.13 67.31)
-		)
-		(stroke
-			(width 0)
-			(type default)
-		)
-	)
-	(wire
-		(pts
 			(xy 129.54 63.5) (xy 134.62 63.5)
 		)
@@
 	(wire
 		(pts
-			(xy 29.21 58.42) (xy 29.21 69.85)
+			(xy 29.21 76.2) (xy 171.45 76.2)
+		)
+		(stroke
+			(width 0)
+			(type default)
+		)
+	)
+	(wire
+		(pts
+			(xy 29.21 58.42) (xy 29.21 76.2)
 		)
 		(stroke
@@
 	(wire
 		(pts
-			(xy 171.45 67.31) (xy 171.45 62.23)
+			(xy 171.45 24.13) (xy 171.45 30.48)
+		)
+		(stroke
+			(width 0)
+			(type default)
+		)
+	)
+	(wire
+		(pts
+			(xy 146.05 52.07) (xy 140.97 52.07)
 		)
 		(stroke
@@
 	(wire
 		(pts
+			(xy 171.45 76.2) (xy 171.45 53.34)
+		)
+		(stroke
+			(width 0)
+			(type default)
+		)
+	)
+	(wire
+		(pts
 			(xy 44.45 52.07) (xy 44.45 58.42)
 		)
@@
 	(wire
 		(pts
+			(xy 140.97 27.94) (xy 146.05 27.94)
+		)
+		(stroke
+			(width 0)
+			(type default)
+		)
+	)
+	(wire
+		(pts
 			(xy 115.57 45.72) (xy 124.46 45.72)
 		)
@@
 	(wire
 		(pts
-			(xy 171.45 21.59) (xy 171.45 43.18)
-		)
-		(stroke
-			(width 0)
-			(type default)
-		)
-	)
-	(wire
-		(pts
 			(xy 44.45 58.42) (xy 59.69 58.42)
 		)
@@
 		(pts
 			(xy 102.87 50.8) (xy 124.46 50.8)
+		)
+		(stroke
+			(width 0)
+			(type default)
+		)
+	)
+	(wire
+		(pts
+			(xy 171.45 33.02) (xy 171.45 43.18)
 		)
 		(stroke
@@
 			)
 		)
-		(property "Value" "4k7"
+		(property "Value" "470"
 			(at 156.21 44.45 90)
 			(effects
@@
 			)
 		)
-		(property "Value" "470"
+		(property "Value" "220"
 			(at 148.59 57.1499 0)
 			(effects
@@
 	(symbol
 		(lib_id "Connector_Generic:Conn_01x02")
-		(at 176.53 59.69 0)
+		(at 176.53 21.59 0)
 		(unit 1)
 		(exclude_from_sim no)
@@
 		(fields_autoplaced yes)
 		(property "Reference" "J3"
-			(at 179.07 59.6899 0)
+			(at 179.07 21.5899 0)
 			(effects
 				(font
@@
 		)
 		(property "Value" "JUMP"
-			(at 179.07 62.2299 0)
+			(at 179.07 24.1299 0)
 			(effects
 				(font
@@
 		)
 		(property "Footprint" "Button_Switch_THT:SW_DIP_SPSTx01_Slide_6.7x4.1mm_W7.62mm_P2.54mm_LowProfile"
-			(at 176.53 59.69 0)
+			(at 176.53 21.59 0)
 			(effects
 				(font
@@
 		)
 		(property "Datasheet" "~"
-			(at 176.53 59.69 0)
+			(at 176.53 21.59 0)
 			(effects
 				(font
@@
 		)
 		(property "Description" "Generic connector, single row, 01x02, script generated (kicad-library-utils/schlib/autogen/connector/)"
-			(at 176.53 59.69 0)
+			(at 176.53 21.59 0)
 			(effects
 				(font
@@
 	(symbol
 		(lib_id "Connector_Generic:Conn_01x02")
-		(at 160.02 72.39 270)
+		(at 176.53 30.48 0)
 		(unit 1)
 		(exclude_from_sim no)
@@
 		(fields_autoplaced yes)
 		(property "Reference" "J2"
-			(at 162.56 71.1199 90)
+			(at 179.07 30.4799 0)
 			(effects
 				(font
@@
 		)
 		(property "Value" "IGNITER"
-			(at 162.56 73.6599 90)
+			(at 179.07 33.0199 0)
 			(effects
 				(font
@@
 		)
 		(property "Footprint" "TerminalBlock_Phoenix:TerminalBlock_Phoenix_MKDS-1,5-2-5.08_1x02_P5.08mm_Horizontal"
-			(at 160.02 72.39 0)
+			(at 176.53 30.48 0)
 			(effects
 				(font
@@
 		)
 		(property "Datasheet" "~"
-			(at 160.02 72.39 0)
+			(at 176.53 30.48 0)
 			(effects
 				(font
@@
 		)
 		(property "Description" "Generic connector, single row, 01x02, script generated (kicad-library-utils/schlib/autogen/connector/)"
-			(at 160.02 72.39 0)
-			(effects
-				(font
+			(at 176.53 30.48 0)
+			(effects
+				(font

Commit message: finalizada com order para JCLPCB
Parts:
- removed D3: LED, LED_THT:LED_D5.0mm, symbol Device:LED
- added D1: LED, LED_THT:LED_D5.0mm, symbol Device:LED
- added J4: ON, Button_Switch_THT:SW_DIP_SPSTx01_Slide_6.7x4.1mm_W7.62mm_P2.54mm_LowProfile, symbol Connector_Generic:Conn_01x02
- added Q1: BC548, Package_TO_SOT_THT:TO-92L_Inline_Wide, symbol Transistor_BJT:BC548
- added R8: 220, Resistor_THT:R_Axial_DIN0204_L3.6mm_D1.6mm_P5.08mm_Horizontal, symbol Device:R
- added unit 2 of U2
- J2: value IGNITER -> TRIGGER
- J3: value JUMP -> READY
- R5: value 220 -> 470
- R6, R7: footprint OptoDevice:R_LDR_5.1x4.3mm_P3.4mm_Vertical -> Connector_PinHeader_2.54mm:PinHeader_1x02_P2.54mm_Vertical
Connections:
- net GND: now also Q1.3 (E)
- net VCC: now also R8.1; no longer R5.1
- net at R5.2: now also Q1.2 (B)
- net at R2.1, R7.1, U2.2 (-): now also U2.5 (+)
- net at R1.1, R6.1, U2.3 (+): now also U2.6 (-)
- net at C1.1, J3.1 (Pin_1), U1.1 (VI): now also J4.1 (Pin_1); no longer J1.1 (Pin_1)
- new net: D1.2 (A), R8.2
- new net: R5.1, U2.7
- new net: J1.1 (Pin_1), J4.2 (Pin_2)
- new net: D1.1 (K), Q1.1 (C)
